Commit message: 04/10 Feat: add jini amp set

File: source/robot_lab/data/Robots/jini/jini.urdf (robot description, URDF)
Before this commit: robot my_robot, 11 links, 10 joints
Links:
- removed link JiNi-Left-Link-1
- removed link JiNi-Left-Link-2
- removed link JiNi-Left-Link-3
- removed link JiNi-Left-Link-4
- removed link JiNi-Left-Link-5
- removed link JiNi-Right-Link-1
- removed link JiNi-Right-Link-2
- removed link JiNi-Right-Link-3
- removed link JiNi-Right-Link-4
- removed link JiNi-Right-Link-5
- added link JiNi_Left_Link_1, mass 1.15155; visual mesh filename=meshes/JiNi_Left_Link_1.STL scale=0.001 0.001 0.001
- added link JiNi_Left_Link_2, mass 0.76315; visual mesh filename=meshes/JiNi_Left_Link_2.STL scale=0.001 0.001 0.001
- added link JiNi_Left_Link_3, mass 1.55469; visual mesh filename=meshes/JiNi_Left_Link_3.STL scale=0.001 0.001 0.001
- added link JiNi_Left_Link_4, mass 0.90055; visual mesh filename=meshes/JiNi_Left_Link_4.STL scale=0.001 0.001 0.001
- added link JiNi_Left_Link_5, mass 0.239; collision sphere radius=0.0020; collision sphere radius=0.0020
- added link JiNi_Right_Link_1, mass 1.15155; visual mesh filename=meshes/JiNi_Right_Link_1.STL scale=0.001 0.001 0.001
- added link JiNi_Right_Link_2, mass 0.76315; visual mesh filename=meshes/JiNi_Right_Link_2.STL scale=0.001 0.001 0.001
- added link JiNi_Right_Link_3, mass 1.55469; visual mesh filename=meshes/JiNi_Right_Link_3.STL scale=0.001 0.001 0.001
- added link JiNi_Right_Link_4, mass 0.90055; visual mesh filename=meshes/JiNi_Right_Link_4.STL scale=0.001 0.001 0.001
- added link JiNi_Right_Link_5, mass 0.239; collision sphere radius=0.0020; collision sphere radius=0.0020
- link base_link: geometry visual mesh filename=meshes/JiNi_Lower_Body_Base.STL scale=0.001 0.001 0.001
Joints:
- removed joint Left-Ankle-Pitch
- removed joint Left-Hip-Pitch
- removed joint Left-Hip-Roll
- removed joint Left-Hip-Yaw
- removed joint Left-Knee-Pitch
- removed joint Right-Ankle-Pitch
- removed joint Right-Hip-Pitch
- removed joint Right-Hip-Roll
- removed joint Right-Hip-Yaw
- removed joint Right-Knee-Pitch
- added joint Left_Ankle_Pitch: type revolute, parent JiNi_Left_Link_4, child JiNi_Left_Link_5, origin xyz=0 0.0485 -0.2 rpy=0.0000 0.0000 0.0000, axis 0 1 0, limit lower=-3.1416 upper=3.1416 effort=10 velocity=1
- added joint Left_Hip_Pitch: type revolute, parent JiNi_Left_Link_2, child JiNi_Left_Link_3, origin xyz=0.0765 0.0015 0 rpy=0.0000 0.0000 0.0000, axis 0 1 0, limit lower=-3.1416 upper=3.1416 effort=10 velocity=1
- added joint Left_Hip_Roll: type revolute, parent JiNi_Left_Link_1, child JiNi_Left_Link_2, origin xyz=-0.0105 0 -0.0815 rpy=0.0000 0.0000 0.0000, axis 1 0 0, limit lower=-3.1416 upper=3.1416 effort=10 velocity=1
- added joint Left_Hip_Yaw: type revolute, parent base_link, child JiNi_Left_Link_1, origin xyz=0 0.06 -0.0295 rpy=0.0000 0.0000 0.0000, axis 0 0 1, limit lower=-3.1416 upper=3.1416 effort=10 velocity=1
- added joint Left_Knee_Pitch: type revolute, parent JiNi_Left_Link_3, child JiNi_Left_Link_4, origin xyz=0 0.0625 -0.2 rpy=0.0000 0.0000 0.0000, axis 0 1 0, limit lower=-3.1416 upper=3.1416 effort=10 velocity=1
- added joint Right_Ankle_Pitch: type revolute, parent JiNi_Right_Link_4, child JiNi_Right_Link_5, origin xyz=0 -0.0485 -0.2 rpy=0.0000 0.0000 0.0000, axis 0 1 0, limit lower=-3.1416 upper=3.1416 effort=10 velocity=1
- added joint Right_Hip_Pitch: type revolute, parent JiNi_Right_Link_2, child JiNi_Right_Link_3, origin xyz=0.0765 -0.0015 0 rpy=0.0000 0.0000 0.0000, axis 0 1 0, limit lower=-3.1416 upper=3.1416 effort=10 velocity=1
- added joint Right_Hip_Roll: type revolute, parent JiNi_Right_Link_1, child JiNi_Right_Link_2, origin xyz=-0.0105 0 -0.0815 rpy=0.0000 0.0000 0.0000, axis 1 0 0, limit lower=-3.1416 upper=3.1416 effort=10 velocity=1
- added joint Right_Hip_Yaw: type revolute, parent base_link, child JiNi_Right_Link_1, origin xyz=0 -0.06 -0.0295 rpy=0.0000 0.0000 0.0000, axis 0 0 1, limit lower=-3.1416 upper=3.1416 effort=10 velocity=1
- added joint Right_Knee_Pitch: type revolute, parent JiNi_Right_Link_3, child JiNi_Right_Link_4, origin xyz=0 -0.0625 -0.2 rpy=0.0000 0.0000 0.0000, axis 0 1 0, limit lower=-3.1416 upper=3.1416 effort=10 velocity=1
